File: hardware/marlin-486-proto/marlin-486-proto.kicad_pcb (KiCad board)
At the start: 2 copper layers, 21 parts, among them J1 Conn_01x03, U1 AM486DX, U2 EPM240T100, U3 AS6C4008-55PCN, U4 AS6C4008-55PCN, U5 AS6C4008-55PCN, U6 AS6C4008-55PCN

Commit message: Add 16C550 symbol
Parts:
- added J2: Conn_02x05_Odd_Even, Connector_IDC:IDC-Header_2x05_P2.54mm_Vertical, F.Cu at (-39.8, 101.9)
- added R15: 4k7, Resistor_THT:R_Axial_DIN0207_L6.3mm_D2.5mm_P7.62mm_Horizontal, F.Cu at (-31.5, 97.8)
- added R16: 4k7, Resistor_THT:R_Axial_DIN0207_L6.3mm_D2.5mm_P7.62mm_Horizontal, F.Cu at (-31.5, 101.8)
- added R17: 4k7, Resistor_THT:R_Axial_DIN0207_L6.3mm_D2.5mm_P7.62mm_Horizontal, F.Cu at (-31.5, 105.9)
- added R18: 4k7, Resistor_THT:R_Axial_DIN0207_L6.3mm_D2.5mm_P7.62mm_Horizontal, F.Cu at (-31.5, 109.9)
- added U7: 16C550, Package_LCC:PLCC-44_THT-Socket, F.Cu at (49.4, 90.0)
- added X1: 1.8432 MHz, Oscillator:Oscillator_DIP-8, F.Cu at (-17.2, 86.2)
- U2: moved to B.Cu
- moved U6 97.1 mm to (100.9, 73.1)
- moved U5 97.1 mm to (81.5, 73.1)
- moved J1 91.7 mm to (-31.6, 18.4)
- moved R1 91.7 mm to (-43.1, 18.1)
- moved R10 91.7 mm to (-43.1, 54.5)
- moved R11 91.7 mm to (-43.1, 58.6)
- moved R12 91.7 mm to (-43.1, 62.6)
- moved R13 91.7 mm to (-43.1, 66.7)
- moved R14 91.7 mm to (-43.1, 70.7)
- moved R2 91.7 mm to (-43.1, 22.1)
- moved R3 91.7 mm to (-43.1, 26.2)
- moved R4 91.7 mm to (-43.1, 30.2)
- moved R5 91.7 mm to (-43.1, 34.3)
- moved R6 91.7 mm to (-43.1, 38.3)
- moved R7 91.7 mm to (-43.1, 42.4)
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Connections:
- U2 pad 1: unconnected-(U2-IO2_1-Pad1) -> D0
- U2 pad 100: unconnected-(U2-IO2_100-Pad100) -> A31
- U2 pad 15: unconnected-(U2-IO1_15-Pad15) -> WR
- U2 pad 16: unconnected-(U2-IO1_16-Pad16) -> INT
- U2 pad 17: unconnected-(U2-IO1_17-Pad17) -> NMI
- U2 pad 18: unconnected-(U2-IO1_18-Pad18) -> RESET
- U2 pad 19: unconnected-(U2-IO1_19-Pad19) -> /ADS
- U2 pad 2: unconnected-(U2-IO1_2-Pad2) -> /RESET
- U2 pad 20: unconnected-(U2-IO1_20-Pad20) -> /BS8
- U2 pad 21: unconnected-(U2-IO1_21-Pad21) -> /BS16
- U2 pad 22: unconnected-(U2-TMS-Pad22) -> TMS
- U2 pad 23: unconnected-(U2-TDI-Pad23) -> TDI
- U2 pad 24: unconnected-(U2-TCK-Pad24) -> TCK
- U2 pad 25: unconnected-(U2-TDO-Pad25) -> TDO
- U2 pad 26: unconnected-(U2-IO1_26-Pad26) -> /RDY
- U2 pad 27: unconnected-(U2-IO1_27-Pad27) -> /CS_SRAM0
- U2 pad 28: unconnected-(U2-IO1_28-Pad28) -> /CS_SRAM1
- U2 pad 29: unconnected-(U2-IO1_29-Pad29) -> /CS_SRAM2
- U2 pad 3: unconnected-(U2-IO1_3-Pad3) -> /BE0
- U2 pad 30: unconnected-(U2-IO1_30-Pad30) -> /CS_SRAM3
- U2 pad 33: unconnected-(U2-IO1_33-Pad33) -> A2
- U2 pad 34: unconnected-(U2-IO1_34-Pad34) -> A3
- U2 pad 35: unconnected-(U2-IO1_35-Pad35) -> A4
- U2 pad 36: unconnected-(U2-IO1_36-Pad36) -> A5
- U2 pad 37: unconnected-(U2-IO1_37-Pad37) -> A6
- U2 pad 38: unconnected-(U2-IO1_38-Pad38) -> A7
- U2 pad 39: unconnected-(U2-IO1_39-Pad39) -> A8
- U2 pad 4: unconnected-(U2-IO1_4-Pad4) -> /BE1
- U2 pad 40: unconnected-(U2-IO1_40-Pad40) -> A9
- U2 pad 41: unconnected-(U2-IO1_41-Pad41) -> A10
- U2 pad 42: unconnected-(U2-IO1_42-Pad42) -> A11
- U2 pad 47: unconnected-(U2-IO1_47-Pad47) -> A12
- U2 pad 48: unconnected-(U2-IO1_48-Pad48) -> A13
- U2 pad 49: unconnected-(U2-IO1_49-Pad49) -> A14
- U2 pad 5: unconnected-(U2-IO1_5-Pad5) -> /BE2
- U2 pad 50: unconnected-(U2-IO1_50-Pad50) -> A15
- U2 pad 52: unconnected-(U2-IO2_52-Pad52) -> D1
- U2 pad 53: unconnected-(U2-IO2_53-Pad53) -> D2
- U2 pad 54: unconnected-(U2-IO2_54-Pad54) -> D3
- U2 pad 55: unconnected-(U2-IO2_55-Pad55) -> D4
- U2 pad 56: unconnected-(U2-IO2_56-Pad56) -> D5
- U2 pad 57: unconnected-(U2-IO2_57-Pad57) -> D6
- U2 pad 58: unconnected-(U2-IO2_58-Pad58) -> D7
- U2 pad 6: unconnected-(U2-IO1_6-Pad6) -> /BE3
- U2 pad 61: unconnected-(U2-IO2_61-Pad61) -> D8
- U2 pad 66: unconnected-(U2-IO2_66-Pad66) -> D9
- U2 pad 67: unconnected-(U2-IO2_67-Pad67) -> D10
- U2 pad 68: unconnected-(U2-IO2_68-Pad68) -> D11
- U2 pad 69: unconnected-(U2-IO2_69-Pad69) -> D12
- U2 pad 7: unconnected-(U2-IO1_7-Pad7) -> MIO
- U2 pad 70: unconnected-(U2-IO2_70-Pad70) -> D13
- U2 pad 71: unconnected-(U2-IO2_71-Pad71) -> D14
- U2 pad 72: unconnected-(U2-IO2_72-Pad72) -> D15
- U2 pad 73: unconnected-(U2-IO2_73-Pad73) -> D16
- U2 pad 74: unconnected-(U2-IO2_74-Pad74) -> D17
- U2 pad 75: unconnected-(U2-IO2_75-Pad75) -> D18
- U2 pad 76: unconnected-(U2-IO2_76-Pad76) -> D19
- U2 pad 77: unconnected-(U2-IO2_77-Pad77) -> D20
- U2 pad 78: unconnected-(U2-IO2_78-Pad78) -> D21
- U2 pad 8: unconnected-(U2-IO1_8-Pad8) -> DC
- U2 pad 81: unconnected-(U2-IO2_81-Pad81) -> D22
- U2 pad 82: unconnected-(U2-IO2_82-Pad82) -> D23
- U2 pad 83: unconnected-(U2-IO2_83-Pad83) -> D24
- U2 pad 84: unconnected-(U2-IO2_84-Pad84) -> D25
- U2 pad 85: unconnected-(U2-IO2_85-Pad85) -> D26
- U2 pad 86: unconnected-(U2-IO2_86-Pad86) -> D27
- U2 pad 87: unconnected-(U2-IO2_87-Pad87) -> D28
- U2 pad 88: unconnected-(U2-IO2_88-Pad88) -> D29
- U2 pad 89: unconnected-(U2-IO2_89-Pad89) -> D30
- U2 pad 90: unconnected-(U2-IO2_90-Pad90) -> D31
- U2 pad 97: unconnected-(U2-IO2_97-Pad97) -> A28
- U2 pad 98: unconnected-(U2-IO2_98-Pad98) -> A29
- U2 pad 99: unconnected-(U2-IO2_99-Pad99) -> A30
- U3 pad 24: unconnected-(U3-OE#-Pad24) -> GND
- U3 pad 29: unconnected-(U3-WE#-Pad29) -> /WR
- U4 pad 24: unconnected-(U4-OE#-Pad24) -> GND
- U4 pad 29: unconnected-(U4-WE#-Pad29) -> /WR
- U5 pad 24: unconnected-(U5-OE#-Pad24) -> GND
- U5 pad 29: unconnected-(U5-WE#-Pad29) -> /WR
- U6 pad 24: unconnected-(U6-OE#-Pad24) -> GND
- U6 pad 29: unconnected-(U6-WE#-Pad29) -> /WR
Other:
- board outline added: 100 x 100 mm
